Commit message: updated student modell

File: catkin_ws/src/udacity_bot/urdf/udacity_bot_chris.xacro (robot description, xacro)
@@ -24,6 +24,5 @@
       <origin xyz="0 0 0" rpy=" 0 0 0"/>
       <geometry>
-        <cylinder radius=".3" length=".1"/>
-        <box size=".4 .2 .1"/>
+        <cylinder radius=".25" length=".1"/>
       </geometry>
     </collision>
@@ -31,5 +30,5 @@
       <origin xyz="0 0 0" rpy=" 0 0 0"/>
       <geometry>
-        <cylinder radius=".3" length=".1"/>
+        <cylinder radius=".25" length=".1"/>
       </geometry>
     </visual>
@@ -56,4 +55,16 @@
       <geometry>
         <sphere radius="0.05"/>
+      </geometry>
+    </visual>
+    <collision name='laser_sockel_collision'>
+      <origin xyz="0 0 0.05" rpy=" 0 0 0"/>
+      <geometry>
+        <box size=".1 .1 .1"/>
+      </geometry>
+    </collision>
+    <visual name='laser_sockel_visual'>
+      <origin xyz="0 0 0.05" rpy=" 0 0 0"/>
+      <geometry>
+      	<box size=".1 .1 .1"/>
       </geometry>
     </visual>
@@ -147,5 +158,5 @@
   </link>
   <joint type="fixed" name="camera_joint">
-    <origin xyz="0.2 0 0" rpy="0 0 0"/>
+    <origin xyz="0.25 0 0" rpy="0 0 0"/>
     <child link="camera"/>
     <parent link="chassis"/>
@@ -177,5 +188,5 @@
   </link>
   <joint type="fixed" name="hokuyo_joint">
-    <origin xyz="0.15 0 0.1" rpy="0 0 0"/>
+    <origin xyz="0 0 0.15" rpy="0 0 0"/>
     <child link="hokuyo"/>
     <parent link="chassis"/>
